Commit message: [checkpoint] generated urdf for 'leonardo', removed some temp files

File: src/gen3_7dof/config/kortex_description/robots/gen3_leonardo.xacro (robot description, xacro)
@@ -45,5 +45,5 @@
         fake_sensor_commands="$(arg fake_sensor_commands)"
         use_external_cable="$(arg use_external_cable)" >
-        <origin xyz="0 0 0" rpy="0 0 0" />  <!-- position robot in the world -->
+        <origin xyz="0 -0.058 0.232548" rpy="-1.5708 0 0" />  <!-- position robot in the world -->
     </xacro:load_robot>
 </robot>

File: src/gen3_7dof/config/kortex_description/robots/leonardo.urdf (robot description, URDF)
Before this commit: robot gen3, 11 links, 10 joints
Joints:
- joint base_joint: origin xyz=0 0 0 rpy=0 0 0 -> xyz=0 -0.058 0.232548 rpy=-1.5708 0 0
